File: Schemat - mata/V5.brd (EAGLE design)
At the start: 126 x 84 mm, 21 parts, among them J1 F-1X04-SIP-100-32, X1 RASPI_GPIO_B+#_PIN

Commit message: aktualizacja schematów
Parts:
- removed SV1: (no value), con-lstb:MA08-1
Connections:
- net N$1: no longer SV1.1
- net N$19: no longer SV1.4
- net N$2: no longer SV1.2
- net N$3: no longer SV1.3
- net N$5: no longer SV1.8
- net N$6: no longer SV1.7
- net N$7: no longer SV1.6
- net N$8: no longer SV1.5
Routing:
- net N$1: track 202.9 -> 123.5 mm, vias 1 -> 0
- net N$10: track 53.2 -> 102.2 mm, vias 0 -> 1
- net N$8: track 222.7 -> 175.1 mm, vias 2 -> 1
- net N$2: track 189.7 -> 145.0 mm
- net N$6: track 214.2 -> 170.4 mm, vias 0 -> 1
- net N$7: track 214.7 -> 173.7 mm, vias 2 -> 0
- net N$3: track 175.2 -> 135.8 mm, vias 1 -> 0
- net N$5: track 162.0 -> 130.9 mm
- net N$9: track 74.2 -> 99.6 mm, vias 0 -> 1
- net N$16: track 63.4 -> 75.3 mm
- net N$19: track 184.0 -> 173.3 mm, vias 1 -> 2
- net N$11: track 70.9 -> 72.9 mm
Other:
- board text added: "Mamma mia!"
- board text added: "Robot porusza sie jak zmija!"
