File: Schemat - mata/V5.sch (EAGLE design)
At the start: 21 parts, among them J1 F-1X04-SIP-100-32, X1 RASPI_GPIO_B+#_PIN

Commit message: aktualizacja schematów
Parts:
- removed SV1: (no value), con-lstb:MA08-1
Connections:
- net N$1: no longer SV1.1
- net N$19: no longer SV1.4
- net N$2: no longer SV1.2
- net N$3: no longer SV1.3
- net N$5: no longer SV1.8
- net N$6: no longer SV1.7
- net N$7: no longer SV1.6
- net N$8: no longer SV1.5
Changed lines of the file:
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@@
 <part name="S17" library="switch-omron" library_urn="urn:adsk.eagle:library:377" deviceset="40-XX" device="" package3d_urn="urn:adsk.eagle:package:27483/1"/>
 <part name="S18" library="switch-omron" library_urn="urn:adsk.eagle:library:377" deviceset="40-XX" device="" package3d_urn="urn:adsk.eagle:package:27483/1"/>
-<part name="SV1" library="con-lstb" library_urn="urn:adsk.eagle:library:162" deviceset="MA08-1" device="" package3d_urn="urn:adsk.eagle:package:8343/1"/>
 <part name="J1" library="con-headers-jp" deviceset="F-1X04-" device="SIP-100-32"/>
 <part name="X1" library="raspberrypi_bastelstube_v13" deviceset="RASPI_GPIO_B+#" device="_PIN"/>
@@
 <attribute name="NAME" x="-8.89" y="-20.32" size="1.778" layer="95" rot="R90"/>
 <attribute name="VALUE" x="-6.35" y="-14.605" size="1.778" layer="96" rot="R90"/>
-</instance>
-<instance part="SV1" gate="1" x="35.56" y="114.3" smashed="yes" rot="R270">
-<attribute name="VALUE" x="22.86" y="115.57" size="1.778" layer="96" rot="R270"/>
-<attribute name="NAME" x="49.022" y="115.57" size="1.778" layer="95" rot="R270"/>
 </instance>
 <instance part="J1" gate="G$1" x="111.76" y="-20.32" smashed="yes">
@@
 <wire x1="2.54" y1="88.9" x2="2.54" y2="93.98" width="0.8128" layer="91"/>
 <wire x1="2.54" y1="93.98" x2="27.94" y2="93.98" width="0.8128" layer="91"/>
-<pinref part="SV1" gate="1" pin="1"/>
-<wire x1="27.94" y1="93.98" x2="27.94" y2="106.68" width="0.8128" layer="91"/>
-<wire x1="27.94" y1="106.68" x2="27.94" y2="129.54" width="0.8128" layer="91"/>
+<wire x1="27.94" y1="93.98" x2="27.94" y2="129.54" width="0.8128" layer="91"/>
 <wire x1="27.94" y1="129.54" x2="129.54" y2="129.54" width="0.8128" layer="91"/>
 <wire x1="129.54" y1="129.54" x2="129.54" y2="33.02" width="0.8128" layer="91"/>
-<junction x="27.94" y="106.68"/>
 <wire x1="129.54" y1="33.02" x2="154.94" y2="33.02" width="0.8128" layer="91"/>
 <pinref part="X1" gate="G$1" pin="GPIO04"/>
@@
 <wire x1="27.94" y1="91.44" x2="30.48" y2="91.44" width="0.8128" layer="91"/>
 <junction x="27.94" y="88.9"/>
-<pinref part="SV1" gate="1" pin="2"/>
-<wire x1="30.48" y1="91.44" x2="30.48" y2="106.68" width="0.8128" layer="91"/>
-<wire x1="30.48" y1="106.68" x2="30.48" y2="127" width="0.8128" layer="91"/>
+<wire x1="30.48" y1="91.44" x2="30.48" y2="127" width="0.8128" layer="91"/>
 <wire x1="30.48" y1="127" x2="101.6" y2="127" width="0.8128" layer="91"/>
 <wire x1="101.6" y1="127" x2="101.6" y2="-2.54" width="0.8128" layer="91"/>
-<junction x="30.48" y="106.68"/>
 <wire x1="101.6" y1="-2.54" x2="200.66" y2="-2.54" width="0.8128" layer="91"/>
 <wire x1="200.66" y1="-2.54" x2="200.66" y2="58.42" width="0.8128" layer="91"/>
@@
 <junction x="48.26" y="88.9"/>
 <wire x1="48.26" y1="91.44" x2="33.02" y2="91.44" width="0.8128" layer="91"/>
-<pinref part="SV1" gate="1" pin="3"/>
-<wire x1="33.02" y1="91.44" x2="33.02" y2="106.68" width="0.8128" layer="91"/>
-<wire x1="33.02" y1="106.68" x2="33.02" y2="124.46" width="0.8128" layer="91"/>
+<wire x1="33.02" y1="91.44" x2="33.02" y2="124.46" width="0.8128" layer="91"/>
 <wire x1="33.02" y1="124.46" x2="104.14" y2="124.46" width="0.8128" layer="91"/>
 <wire x1="104.14" y1="124.46" x2="104.14" y2="35.56" width="0.8128" layer="91"/>
-<junction x="33.02" y="106.68"/>
 <wire x1="104.14" y1="35.56" x2="86.36" y2="35.56" width="0.8128" layer="91"/>
 <wire x1="86.36" y1="35.56" x2="86.36" y2="86.36" width="0.8128" layer="91"/>
@@
 <junction x="71.12" y="0"/>
 <wire x1="83.82" y1="104.14" x2="45.72" y2="104.14" width="0.8128" layer="91"/>
-<pinref part="SV1" gate="1" pin="8"/>
-<wire x1="45.72" y1="104.14" x2="45.72" y2="106.68" width="0.8128" layer="91"/>
 <wire x1="96.52" y1="5.08" x2="96.52" y2="134.62" width="0.8128" layer="91"/>
 <wire x1="96.52" y1="134.62" x2="45.72" y2="134.62" width="0.8128" layer="91"/>
-<wire x1="45.72" y1="134.62" x2="45.72" y2="106.68" width="0.8128" layer="91"/>
-<junction x="45.72" y="106.68"/>
+<wire x1="45.72" y1="134.62" x2="45.72" y2="104.14" width="0.8128" layer="91"/>
 <wire x1="96.52" y1="5.08" x2="157.48" y2="5.08" width="0.8128" layer="91"/>
 <pinref part="X1" gate="G$1" pin="GPIO23"/>
@@
 <wire x1="71.12" y1="25.4" x2="71.12" y2="27.94" width="0.8128" layer="91"/>
 <junction x="48.26" y="25.4"/>
-<pinref part="SV1" gate="1" pin="7"/>
-<wire x1="43.18" y1="106.68" x2="43.18" y2="101.6" width="0.8128" layer="91"/>
 <wire x1="43.18" y1="101.6" x2="81.28" y2="101.6" width="0.8128" layer="91"/>
 <wire x1="81.28" y1="101.6" x2="81.28" y2="25.4" width="0.8128" layer="91"/>
@@
 <junction x="71.12" y="25.4"/>
 <wire x1="132.08" y1="132.08" x2="43.18" y2="132.08" width="0.8128" layer="91"/>
-<wire x1="43.18" y1="132.08" x2="43.18" y2="106.68" width="0.8128" layer="91"/>
-<junction x="43.18" y="106.68"/>
+<wire x1="43.18" y1="132.08" x2="43.18" y2="101.6" width="0.8128" layer="91"/>
 <wire x1="132.08" y1="132.08" x2="132.08" y2="96.52" width="0.8128" layer="91"/>
 <pinref part="X1" gate="G$1" pin="GPIO22"/>
@@
 <wire x1="71.12" y1="50.8" x2="71.12" y2="53.34" width="0.8128" layer="91"/>
 <junction x="48.26" y="50.8"/>
-<pinref part="SV1" gate="1" pin="6"/>
-<wire x1="40.64" y1="106.68" x2="40.64" y2="99.06" width="0.8128" layer="91"/>
 <wire x1="40.64" y1="99.06" x2="78.74" y2="99.06" width="0.8128" layer="91"/>
 <wire x1="78.74" y1="99.06" x2="78.74" y2="53.34" width="0.8128" layer="91"/>
@@
 <wire x1="40.64" y1="116.84" x2="124.46" y2="116.84" width="0.8128" layer="91"/>
 <wire x1="124.46" y1="116.84" x2="124.46" y2="35.56" width="0.8128" layer="91"/>
-<wire x1="40.64" y1="106.68" x2="40.64" y2="116.84" width="0.8128" layer="91"/>
-<junction x="40.64" y="106.68"/>
+<wire x1="40.64" y1="99.06" x2="40.64" y2="116.84" width="0.8128" layer="91"/>
 <wire x1="124.46" y1="35.56" x2="152.4" y2="35.56" width="0.8128" layer="91"/>
 <wire x1="152.4" y1="35.56" x2="152.4" y2="68.58" width="0.8128" layer="91"/>
@@
 <wire x1="76.2" y1="78.74" x2="76.2" y2="96.52" width="0.8128" layer="91"/>
 <wire x1="76.2" y1="96.52" x2="38.1" y2="96.52" width="0.8128" layer="91"/>
-<pinref part="SV1" gate="1" pin="5"/>
-<wire x1="38.1" y1="96.52" x2="38.1" y2="106.68" width="0.8128" layer="91"/>
 <wire x1="38.1" y1="119.38" x2="99.06" y2="119.38" width="0.8128" layer="91"/>
 <wire x1="99.06" y1="119.38" x2="99.06" y2="7.62" width="0.8128" layer="91"/>
-<wire x1="38.1" y1="106.68" x2="38.1" y2="119.38" width="0.8128" layer="91"/>
-<junction x="38.1" y="106.68"/>
+<wire x1="38.1" y1="96.52" x2="38.1" y2="119.38" width="0.8128" layer="91"/>
 <wire x1="99.06" y1="7.62" x2="160.02" y2="7.62" width="0.8128" layer="91"/>
 <wire x1="160.02" y1="7.62" x2="160.02" y2="22.86" width="0.8128" layer="91"/>
@@
 <junction x="71.12" y="88.9"/>
 <wire x1="71.12" y1="93.98" x2="35.56" y2="93.98" width="0.8128" layer="91"/>
-<pinref part="SV1" gate="1" pin="4"/>
-<wire x1="35.56" y1="93.98" x2="35.56" y2="106.68" width="0.8128" layer="91"/>
 <wire x1="35.56" y1="121.92" x2="127" y2="121.92" width="0.8128" layer="91"/>
 <wire x1="127" y1="121.92" x2="127" y2="38.1" width="0.8128" layer="91"/>
-<wire x1="35.56" y1="106.68" x2="35.56" y2="121.92" width="0.8128" layer="91"/>
-<junction x="35.56" y="106.68"/>
+<wire x1="35.56" y1="93.98" x2="35.56" y2="121.92" width="0.8128" layer="91"/>
 <wire x1="127" y1="38.1" x2="134.62" y2="38.1" width="0.8128" layer="91"/>
 <wire x1="134.62" y1="38.1" x2="134.62" y2="76.2" width="0.8128" layer="91"/>
