File: Schemat - mata/V6.brd (EAGLE design)
At the start: 126 x 84 mm, 20 parts, among them J1 F-1X04-SIP-100-32, X1 RASPI_GPIO_B+#_PIN

Commit message: aktualizacja schematów
Connections:
- removed net GND_A: X1.6
- removed net N$15 (its old number): J1.1, X1.3
- removed net N$16: J1.2, X1.5
- removed net N$18: J1.3, X1.2
- new net N$12: J1.3, X1.5
- new net N$14: J1.2, X1.6
- new net N$3: J1.1, X1.2
- net N$4: now also X1.3; no longer X1.40
Routing:
- net N$16: track 75.3 -> 0.00 mm
- net N$12: track 0.00 -> 64.0 mm
- net N$15 (its old number): track 62.1 -> 0.00 mm
- net N$3: track 0.00 -> 51.9 mm
- net N$18: track 49.7 -> 0.00 mm
- net N$4: track 11.7 -> 61.0 mm, vias 0 -> 1
- net N$14: track 0.00 -> 45.8 mm
- net N$2: track 145.0 -> 118.5 mm, vias 0 -> 1
- net N$8: track 175.1 -> 194.7 mm, vias 1 -> 2
- net N$9: track 135.8 -> 150.8 mm, vias 0 -> 1
- net N$10: track 102.2 -> 110.3 mm, vias 1 -> 3
- net N$6: track 170.4 -> 166.3 mm
- net N$19: track 173.3 -> 175.9 mm, vias 2 -> 3
- net N$1: track 123.5 -> 125.1 mm
- net N$5: track 130.9 -> 129.6 mm
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