File: Schemat - mata/V6.sch (EAGLE design)
At the start: 20 parts, among them J1 F-1X04-SIP-100-32, X1 RASPI_GPIO_B+#_PIN

Commit message: aktualizacja schematów
Connections:
- removed net N$15 (its old number): J1.1, X1.SDA
- removed net N$16: J1.2, X1.SCL
- removed net N$18: J1.3, X1.5V0A
- new net N$12: J1.3, X1.SCL
- new net N$14: J1.2, X1.GND_A
- new net N$3: J1.1, X1.5V0A
- net N$4: now also X1.SDA; no longer X1.GPIO21
Other:
- moved on the sheet: J1
