File: Schemat - robot/Robot_V6.brd (EAGLE design)
At the start: 160 x 100 mm, 6 parts, among them IC1 786TV, J1 F-1X03-SIP-100-32, J2 F-1X03-SIP-100-32, J3 F-1X02-SIP-100-32

Commit message: aktualizacja schematów
Parts:
- added J4: F-1X02-SIP-100-40, con-headers-jp:SIP-100-02-40
- moved C1 12.7 mm to (11.4, 5.08)
- moved J1 4.58 mm to (12.7, 22.9)
- moved J3 3.81 mm to (14.0, 44.5)
- moved IC1 3.81 mm to (21.6, 6.35)
- moved J2 2.84 mm to (12.7, 33.0)
Connections:
- net N$2: now also J4.1
- net N$9: now also J4.2
Routing:
- net N$1: track 74.9 -> 0.00 mm
- net N$2: track 60.3 -> 67.4 mm
- net N$10: track 19.5 -> 14.3 mm
- net N$9: track 38.2 -> 43.2 mm
- net N$5: track 10.5 -> 8.16 mm
- net N$3: track 10.3 -> 8.13 mm
- net N$4: track 10.2 -> 8.17 mm
- net N$6: track 10.4 -> 9.26 mm
- net N$7: track 10.2 -> 9.17 mm
- net N$8: track 10.2 -> 9.21 mm
Other:
- outline, holes or cut-outs redrawn
- board text added: "A tutaj mamy dol"
- board text added: "Tutaj gora"
